File: rolup.kicad_pcb (KiCad board)
At the start: 2 copper layers, 31.3 x 54.2 mm, 11 parts, among them J1 switch, J2 Screw_Terminal_01x03, J3 bala paiin, J4 k a, J5 k b, J6 Conn_01x07_Pin, J7 5+

Commit message: pcb rol
Routing:
- net GND: track 96.5 -> 98.7 mm
- net Net-(J2-Pin_2): track 50.7 -> 51.7 mm
- net Net-(J5-Pin_1): track 23.9 -> 23.0 mm
- net Net-(J3-Pin_1): track 16.9 -> 16.2 mm
Changed lines of the file:
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@@
 			(outputformat 1)
 			(mirror no)
-			(drillshape 1)
+			(drillshape 0)
 			(scaleselection 1)
 			(outputdirectory "")
@@
 			(pintype "passive")
 		)
-		(pad "2" thru_hole oval
+		(pad "2" thru_hole circle
 			(at 7.62 0 270)
-			(size 1.4 1.4)
+			(size 2 2)
 			(drill 0.7)
 			(layers "*.Cu" "*.Mask")
@@
 			)
 		)
-		(pad "1" thru_hole roundrect
+		(pad "1" thru_hole rect
 			(at 0 0 270)
 			(size 2.4 2.4)
@@
 			(layers "*.Cu" "*.Mask")
 			(remove_unused_layers no)
-			(roundrect_rratio 0.104167)
 			(net 7 "+5C")
 			(pinfunction "Pin_1")
@@
 		(pad "1" thru_hole rect
 			(at 0 0 270)
-			(size 2.8 2.8)
-			(drill 1.4)
+			(size 3 3)
+			(drill 1.5)
 			(layers "*.Cu" "*.Mask")
 			(remove_unused_layers no)
@@
 		(pad "2" thru_hole circle
 			(at 5 0 270)
-			(size 2.8 2.8)
-			(drill 1.4)
+			(size 4 4)
+			(drill 1.5)
 			(layers "*.Cu" "*.Mask")
 			(remove_unused_layers no)
@@
 		(tags "THT terminal block Metz Connect Type011_RT05502HBWC pitch 5mm size 10x10.5mm^2 drill 1.4mm pad 2.8mm")
 		(property "Reference" "J7"
-			(at 2.5 -7.56 360)
+			(at 2.5 -7.56 0)
 			(layer "F.SilkS")
 			(effects
@@
 		)
 		(property "Value" "5+"
-			(at 2.5 5.06 360)
+			(at 2.5 5.06 0)
 			(layer "F.Fab")
 			(effects
@@
 		)
 		(fp_text user "${REFERENCE}"
-			(at 2.5 3.25 360)
+			(at 2.5 3.25 0)
 			(layer "F.Fab")
 			(effects
@@
 		(tags "Resistor Axial_DIN0204 series Axial Horizontal pin pitch 7.62mm 0.167W length 3.6mm diameter 1.6mm")
 		(property "Reference" "R2"
-			(at 3.81 -1.92 360)
+			(at 3.81 -1.92 0)
 			(layer "F.SilkS")
 			(effects
@@
 		)
 		(property "Value" "10 k"
-			(at 3.81 1.92 360)
+			(at 3.81 1.92 0)
 			(layer "F.Fab")
 			(effects
@@
 		)
 		(fp_text user "${REFERENCE}"
-			(at 3.7 0 360)
+			(at 3.7 0 0)
 			(layer "F.Fab")
 			(effects
@@
 		(pad "1" thru_hole circle
 			(at 0 0)
-			(size 1.4 1.4)
+			(size 2 2)
 			(drill 0.7)
 			(layers "*.Cu" "*.Mask")
@@
 			(pintype "passive")
 		)
-		(pad "2" thru_hole oval
+		(pad "2" thru_hole circle
 			(at 7.62 0)
-			(size 1.4 1.4)
+			(size 2 2)
 			(drill 0.7)
 			(layers "*.Cu" "*.Mask")
@@
 		(pad "1" thru_hole rect
 			(at 0 0 270)
-			(size 2.8 2.8)
+			(size 3 3)
 			(drill 1.4)
 			(layers "*.Cu" "*.Mask")
@@
 		(pad "2" thru_hole circle
 			(at 5 0 270)
-			(size 2.8 2.8)
+			(size 4 4)
 			(drill 1.4)
 			(layers "*.Cu" "*.Mask")
@@
 		(pad "3" thru_hole circle
 			(at 10 0 270)
-			(size 2.8 2.8)
+			(size 4 4)
 			(drill 1.4)
 			(layers "*.Cu" "*.Mask")
@@
 	)
 	(segment
+		(start 43.45 69.175)
+		(end 41.3 71.325)
+		(width 2)
+		(layer "B.Cu")
+		(net 1)
+	)
+	(segment
 		(start 44.875 83.475)
 		(end 38.125 83.475)
@@
 	)
 	(segment
-		(start 26.1 108.6)
-		(end 31.15 113.65)
+		(start 37.2 71.325)
+		(end 35.75 72.775)
 		(width 2)
 		(layer "B.Cu")
@@
 	)
 	(segment
-		(start 26.1 92.5)
-		(end 31.15 97.55)
+		(start 35.75 72.775)
+		(end 31.125 72.775)
 		(width 2)
 		(layer "B.Cu")
@@
 	)
 	(segment
-		(start 31.125 72.775)
-		(end 28.1 72.775)
+		(start 26.1 86.325)
+		(end 26.1 92.5)
 		(width 2)
 		(layer "B.Cu")
@@
 	)
 	(segment
-		(start 26.1 92.5)
-		(end 26.1 108.6)
+		(start 31.125 72.775)
+		(end 28.1 72.775)
 		(width 2)
 		(layer "B.Cu")
@@
 	)
 	(segment
-		(start 39.85 72.775)
-		(end 31.125 72.775)
+		(start 26.7 97.55)
+		(end 26.1 96.95)
 		(width 2)
 		(layer "B.Cu")
@@
 	)
 	(segment
-		(start 43.45 69.175)
-		(end 39.85 72.775)
+		(start 28.25 113.65)
+		(end 31.15 113.65)
 		(width 2)
 		(layer "B.Cu")
@@
 	)
 	(segment
-		(start 26.1 81.245)
-		(end 26.1 92.5)
+		(start 26.1 92.5)
+		(end 26.1 111.5)
 		(width 2)
 		(layer "B.Cu")
@@
 	)
 	(segment
-		(start 26.1 81.245)
-		(end 31.14 86.285)
+		(start 41.3 71.325)
+		(end 37.2 71.325)
 		(width 2)
 		(layer "B.Cu")
@@
 	)
 	(segment
+		(start 31.15 97.55)
+		(end 26.7 97.55)
+		(width 3)
+		(layer "B.Cu")
+		(net 1)
+	)
+	(segment
+		(start 26.14 86.285)
+		(end 26.1 86.325)
+		(width 2)
+		(layer "B.Cu")
+		(net 1)
+	)
+	(segment
+		(start 26.1 81.245)
+		(end 26.1 86.325)
+		(width 2)
+		(layer "B.Cu")
+		(net 1)
+	)
+	(segment
 		(start 26.1 74.775)
 		(end 26.1 81.245)
@@
 	)
 	(segment
+		(start 26.1 111.5)
+		(end 28.25 113.65)
+		(width 2)
+		(layer "B.Cu")
+		(net 1)
+	)
+	(segment
+		(start 31.14 86.285)
+		(end 26.14 86.285)
+		(width 2)
+		(layer "B.Cu")
+		(net 1)
+	)
+	(segment
+		(start 26.1 92.5)
+		(end 26.1 96.95)
+		(width 2)
+		(layer "B.Cu")
+		(net 1)
+	)
+	(segment
 		(start 38.2 92.55)
 		(end 31.15 92.55)
@@
 	)
 	(segment
-		(start 42.76 98.465)
-		(end 42 99.225)
+		(start 42 100.4)
+		(end 42 112.1)
 		(width 2)
 		(layer "B.Cu")
@@
 	)
 	(segment
-		(start 42 99.225)
-		(end 42 112.1)
+		(start 43.935 98.465)
+		(end 42 100.4)
 		(width 2)
 		(layer "B.Cu")
@@
 	(segment
 		(start 45.725 98.465)
-		(end 42.76 98.465)
+		(end 43.935 98.465)
 		(width 2)
 		(layer "B.Cu")
@@
 	)
 	(segment
-		(start 28.515 78.66)
-		(end 31.14 81.285)
+		(start 31.14 81.285)
+		(end 29.15 79.295)
 		(width 2)
 		(layer "B.Cu")
@@
 		(start 28.515 77.075)
 		(end 28.515 78.66)
-		(width 2)
+		(width 1.5)
 		(layer "B.Cu")
 		(net 6)
@@
 	)
 	(segment
-		(start 50.725 113.1)
-		(end 48.625 115.2)
+		(start 32.65 108.65)
+		(end 31.15 108.65)
 		(width 2)
 		(layer "B.Cu")
@@
 	)
 	(segment
-		(start 31.325 108.65)
-		(end 31.15 108.65)
+		(start 50.725 113.925)
+		(end 48.825 115.825)
 		(width 2)
 		(layer "B.Cu")
@@
 	)
 	(segment
-		(start 48.625 115.2)
-		(end 37.875 115.2)
+		(start 48.825 115.825)
+		(end 39.825 115.825)
 		(width 2)
 		(layer "B.Cu")
@@
 	)
 	(segment
-		(start 37.875 115.2)
-		(end 31.325 108.65)
+		(start 50.725 85.785)
+		(end 50.725 113.925)
 		(width 2)
 		(layer "B.Cu")
@@
 	)
 	(segment
-		(start 50.725 85.785)
-		(end 50.725 113.1)
+		(start 39.825 115.825)
+		(end 32.65 108.65)
 		(width 2)
 		(layer "B.Cu")

Commit message: file pcb add
Parts:
- J6: footprint Connector_TE-Connectivity:TE_826576-7_1x07_P3.96mm_Vertical -> Connector_JST:JST_EH_B7B-EH-A_1x07_P2.50mm_Vertical
- moved R4 6.35 mm to (50.6, 92.1)
- moved J6 6.19 mm to (46.9, 84.8)
Routing:
- net +5C: track 53.9 -> 65.6 mm
- net Net-(J2-Pin_2): track 51.7 -> 45.5 mm
- net Net-(J4-Pin_1): track 55.1 -> 58.9 mm
- net Net-(J5-Pin_1): track 23.0 -> 25.9 mm
- net GND: track 98.7 -> 101.1 mm
- net Net-(J3-Pin_2): track 10.2 -> 12.4 mm
- net Net-(J3-Pin_1): track 16.2 -> 18.3 mm
- net Net-(J2-Pin_1): track 18.4 -> 19.6 mm
