File: rolup.kicad_pcb (KiCad board)
At the start: 2 copper layers, 31.3 x 54.2 mm, 11 parts, among them J1 switch, J2 Screw_Terminal_01x03, J3 bala paiin, J4 k a, J5 k b, J6 Conn_01x07_Pin, J7 5+

Commit message: pcb
Connections:
- J3 pad 1: Net-(J3-Pin_1) -> Net-(J3-Pin_2)
Changed lines of the file:
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@@
 			(at 0 0 90)
 			(size 1.4 1.4)
-			(drill 0.7)
+			(drill 1)
 			(layers "*.Cu" "*.Mask")
 			(remove_unused_layers no)
@@
 			(at 7.62 0 90)
 			(size 1.4 1.4)
-			(drill 0.7)
+			(drill 1)
 			(layers "*.Cu" "*.Mask")
 			(remove_unused_layers no)
@@
 			(at 0 0 270)
 			(size 2 2)
-			(drill 0.95)
+			(drill 1)
 			(layers "*.Cu" "*.Mask")
 			(remove_unused_layers no)
@@
 			(at 2.5 0 270)
 			(size 2 2)
-			(drill 0.95)
+			(drill 1)
 			(layers "*.Cu" "*.Mask")
 			(remove_unused_layers no)
@@
 			(at 5 0 270)
 			(size 2 2)
-			(drill 0.95)
+			(drill 1)
 			(layers "*.Cu" "*.Mask")
 			(remove_unused_layers no)
@@
 			(at 7.5 0 270)
 			(size 2 2)
-			(drill 0.95)
+			(drill 1)
 			(layers "*.Cu" "*.Mask")
 			(remove_unused_layers no)
@@
 			(at 10 0 270)
 			(size 1.7 1.95)
-			(drill 0.95)
+			(drill 1)
 			(layers "*.Cu" "*.Mask")
 			(remove_unused_layers no)
@@
 			(at 15 0 270)
 			(size 2 2)
-			(drill 0.95)
+			(drill 1)
 			(layers "*.Cu" "*.Mask")
 			(remove_unused_layers no)
@@
 			(at 0 0 270)
 			(size 3 3)
-			(drill 1.5)
+			(drill 1)
 			(layers "*.Cu" "*.Mask")
 			(remove_unused_layers no)
@@
 			(at 5 0 270)
 			(size 4 4)
-			(drill 1.5)
+			(drill 1)
 			(layers "*.Cu" "*.Mask")
 			(remove_unused_layers no)
@@
 			(at 0 0)
 			(size 2.8 2.8)
-			(drill 1.4)
+			(drill 1)
 			(layers "*.Cu" "*.Mask")
 			(remove_unused_layers no)
@@
 			(pintype "passive")
 		)
-		(pad "2" thru_hole circle
+		(pad "1" thru_hole circle
 			(at 5 0)
 			(size 2.8 2.8)
-			(drill 1.4)
+			(drill 1)
 			(layers "*.Cu" "*.Mask")
 			(remove_unused_layers no)
@@
 			(at 0 0 270)
 			(size 3 3)
-			(drill 1.4)
+			(drill 1)
 			(layers "*.Cu" "*.Mask")
 			(remove_unused_layers no)
@@
 			(at 5 0 270)
 			(size 4 4)
-			(drill 1.4)
+			(drill 1)
 			(layers "*.Cu" "*.Mask")
 			(remove_unused_layers no)
@@
 			(at 10 0 270)
 			(size 4 4)
-			(drill 1.4)
+			(drill 1)
 			(layers "*.Cu" "*.Mask")
 			(remove_unused_layers no)
