File: rolup.kicad_sch (KiCad schematic)
At the start: 10 parts, among them J1 switch, J2 phto, J3 bala paiin, J4 k a, J5 k b, J6 Conn_01x10_Pin, J7 k b

Commit message: pcb
Parts:
- removed J2: phto, symbol Connector:Screw_Terminal_01x02
- removed J6: Conn_01x10_Pin, Connector_Wuerth:Wuerth_WR-WTB_64801011622_1x10_P1.50mm_Vertical, symbol Connector:Conn_01x10_Pin
- added J2: Screw_Terminal_01x03, TerminalBlock_MetzConnect:TerminalBlock_MetzConnect_Type011_RT05503HBWC_1x03_P5.00mm_Horizontal, symbol Connector:Screw_Terminal_01x03
- added J6: Conn_01x07_Pin, Connector_TE-Connectivity:TE_826576-7_1x07_P3.96mm_Vertical, symbol Connector:Conn_01x07_Pin
- added R4: 10 k, Resistor_THT:R_Axial_DIN0204_L3.6mm_D1.6mm_P7.62mm_Horizontal, symbol Device:R_Small
- J1: footprint TerminalBlock:TerminalBlock_bornier-2_P5.08mm -> TerminalBlock_MetzConnect:TerminalBlock_MetzConnect_Type011_RT05502HBWC_1x02_P5.00mm_Horizontal
- J3, J4, J5: footprint (none) -> TerminalBlock_MetzConnect:TerminalBlock_MetzConnect_Type011_RT05502HBWC_1x02_P5.00mm_Horizontal
- J7: value k b -> 5+; footprint (none) -> TerminalBlock_MetzConnect:TerminalBlock_MetzConnect_Type011_RT05502HBWC_1x02_P5.00mm_Horizontal
- R1, R2, R3: footprint (none) -> Resistor_THT:R_Axial_DIN0204_L3.6mm_D1.6mm_P7.62mm_Horizontal
Connections:
- net +5C: now also J7.1 (Pin_1), R1.2, R2.2, R3.2, J6.1 (Pin_1); no longer R1.1, R2.1, R3.1
- net GND: now also J7.2 (Pin_2), J2.3 (Pin_3), J6.2 (Pin_2), R4.1
- net at J1.1 (Pin_1): now also R3.1; no longer R1.2
- net at J5.1 (Pin_1): now also R2.1, J6.4 (Pin_4); no longer R3.2
- net at J3.1 (Pin_1): now also J6.6 (Pin_6)
- net at J3.2 (Pin_2): now also J6.7 (Pin_7)
- net at J4.1 (Pin_1): now also R1.1, J6.3 (Pin_3); no longer R2.2
- new net: J2.1 (Pin_1), J6.5 (Pin_5)
Other:
- moved on the sheet: J1, J3, J4, J5, J7, R1, R2

Commit message: file pcb add
Parts:
- J6: footprint Connector_TE-Connectivity:TE_826576-7_1x07_P3.96mm_Vertical -> Connector_JST:JST_EH_B7B-EH-A_1x07_P2.50mm_Vertical
Connections:
- net +5C: now also R4.2
- net GND: no longer R4.1
- net at J2.2 (Pin_2): now also R4.1
Other:
- moved on the sheet: R4
Changed lines of the file:
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@@
-	)
-	(junction
-		(at 36.83 72.39)
-		(diameter 0)
-		(color 0 0 0 0)
 	)
 	(junction
@@
 	(wire
 		(pts
-			(xy 39.37 74.93) (xy 39.37 81.28)
+			(xy 40.64 74.93) (xy 40.64 81.28)
 		)
 		(stroke
@@
 	(wire
 		(pts
-			(xy 36.83 55.88) (xy 36.83 72.39)
-		)
-		(stroke
-			(width 0)
-			(type default)
-		)
-	)
-	(wire
-		(pts
 			(xy 30.48 48.26) (xy 30.48 50.8)
 		)
@@
 	(wire
 		(pts
-			(xy 36.83 72.39) (xy 36.83 83.82)
+			(xy 36.83 55.88) (xy 36.83 83.82)
 		)
 		(stroke
@@
 	(wire
 		(pts
-			(xy 39.37 81.28) (xy 49.53 81.28)
+			(xy 40.64 81.28) (xy 49.53 81.28)
 		)
 		(stroke
@@
 	(wire
 		(pts
-			(xy 39.37 69.85) (xy 35.56 69.85)
+			(xy 40.64 69.85) (xy 35.56 69.85)
 		)
 		(stroke
@@
 	(symbol
 		(lib_id "Device:R_Small")
-		(at 39.37 72.39 90)
+		(at 40.64 72.39 180)
 		(unit 1)
 		(exclude_from_sim no)
@@
 		(fields_autoplaced yes)
 		(property "Reference" "R4"
-			(at 39.37 69.85 90)
-			(effects
-				(font
-					(size 1.27 1.27)
-				)
+			(at 43.18 72.3899 0)
+			(effects
+				(font
+					(size 1.27 1.27)
+				)
+				(justify right)
 			)
 		)
 		(property "Value" "10 k"
-			(at 39.37 69.85 90)
+			(at 38.1 72.39 90)
 			(effects
 				(font
@@
 		)
 		(property "Footprint" "Resistor_THT:R_Axial_DIN0204_L3.6mm_D1.6mm_P7.62mm_Horizontal"
-			(at 39.37 72.39 0)
+			(at 40.64 72.39 0)
 			(effects
 				(font
@@
 		)
 		(property "Datasheet" "~"
-			(at 39.37 72.39 0)
+			(at 40.64 72.39 0)
 			(effects
 				(font
@@
 		)
 		(property "Description" "Resistor, small symbol"
-			(at 39.37 72.39 0)
+			(at 40.64 72.39 0)
 			(effects
 				(font
@@
 			)
 		)
-		(property "Footprint" "Connector_TE-Connectivity:TE_826576-7_1x07_P3.96mm_Vertical"
+		(property "Footprint" "Connector_JST:JST_EH_B7B-EH-A_1x07_P2.50mm_Vertical"
 			(at 19.05 60.96 0)
 			(effects
